File: Fixteen.kicad_pcb (KiCad board)
At the start: 2 copper layers, 33.5 x 62.7 mm, 15 parts, among them J1 TED_SOCKET, J2 RAM_SELECTOR, U1 MOS_7360_TED, U2 74LS257, U3 74LS257, U4 4464, U5 4464, U6 DT1042, U7 DT1042

Commit message: Cut corner, for the thing to hopefully fit with MCes's CPU4C16 - Untested!
Parts:
- added J99: OSHW_LOGO, Symbol:OSHW-Logo_5.7x6mm_Copper, B.Cu at (131.1, 131.8)
- moved R2 1.62 mm to (146.8, 131.8), turned to 270 degrees
Routing:
- net d0: track 37.4 -> 35.2 mm
- net d1: track 39.8 -> 37.7 mm
- net VCC: track 135.2 -> 134.7 mm
- net GND: vias 8 -> 9
Other:
- board size 33.5 x 62.7 mm -> 33.8 x 62.7 mm
