File: Fixteen.sch (KiCad schematic (older format))
At the start: 8 parts, among them J1 TED_SOCKET, J2 RAM_SELECTOR, J99 OSHW_LOGO, U1 MOS_7360_TED, U6 DT1042, U7 DT1042

Commit message: Cut corner, for the thing to hopefully fit with MCes's CPU4C16 - Untested!
Parts:
- J99: footprint Symbol:OSHW-Logo_7.5x8mm_Copper -> Symbol:OSHW-Logo_5.7x6mm_Copper
Changed lines of the file:
@@
 F 0 "J99" H 11168 6531 50  0000 C CNN
 F 1 "OSHW_LOGO" H 11168 6440 50  0000 C CNN
-F 2 "Symbol:OSHW-Logo_7.5x8mm_Copper" H 11060 6350 50  0001 C CNN
+F 2 "Symbol:OSHW-Logo_5.7x6mm_Copper" H 11060 6350 50  0001 C CNN
 F 3 "~" H 11060 6350 50  0001 C CNN
 	1    11060 6350
