File: ram.sch (KiCad schematic (older format))
At the start: 8 parts, among them U2 74LS257, U3 74LS257, U4 4464, U5 4464

Commit message: Redo connections as they are on OpenC16RamExpansion V2 did not work :(
Connections:
- net a0: now also U2.3 (B1); no longer U2.6 (B2)
- net a1: now also U2.6 (B2); no longer U2.3 (B1)
- net a10: now also U2.14 (A4); no longer U2.11 (A3)
- net a11: now also U3.2 (A1); no longer U2.5 (A2)
- net a12: now also U3.5 (A2); no longer U3.14 (A4)
- net a13: now also U3.11 (A3); no longer U3.2 (A1)
- net a14: now also U3.14 (A4); no longer U3.5 (A2)
- net a15: now also U2.2 (A1); no longer U3.11 (A3)
- net a4: now also U3.3 (B1); no longer U3.13 (B4)
- net a5: now also U3.6 (B2); no longer U3.3 (B1)
- net a6: now also U3.10 (B3); no longer U3.6 (B2)
- net a7: now also U3.13 (B4); no longer U3.10 (B3)
- net a8: now also U2.5 (A2); no longer U2.14 (A4)
- net a9: now also U2.11 (A3); no longer U2.2 (A1)
- net m1: now also U2.7 (Y2); no longer U3.4 (Y1)
- net m2: now also U2.9 (Y3); no longer U3.12 (Y4)
- net m3: now also U2.12 (Y4); no longer U3.7 (Y2)
- net m4: now also U3.4 (Y1); no longer U2.9 (Y3)
- net m5: now also U3.7 (Y2); no longer U2.7 (Y2)
- net m6: now also U3.9 (Y3); no longer U2.12 (Y4)
- net m7: now also U3.12 (Y4); no longer U3.9 (Y3)
Changed lines of the file:
@@
 Sheet 2 2
 Title "Fixteen"
-Date "2020-11-28"
-Rev "2git"
+Date "2020-12-21"
+Rev "3git"
 Comp "SukkoPera"
 Comment1 "Licensed under CERN OHL v.1.2"
@@
 	1930 4655 2030 4755
 Text Label 2230 2205 0    60   ~ 0
+a15
+Text Label 2230 2305 0    60   ~ 0
+a0
+Text Label 2230 2455 0    60   ~ 0
+a8
+Text Label 2230 2555 0    60   ~ 0
+a1
+Text Label 2230 2705 0    60   ~ 0
 a9
-Text Label 2230 2305 0    60   ~ 0
-a1
-Text Label 2230 2455 0    60   ~ 0
-a11
-Text Label 2230 2555 0    60   ~ 0
-a0
-Text Label 2230 2705 0    60   ~ 0
-a10
 Text Label 2230 2805 0    60   ~ 0
 a2
 Text Label 2230 2955 0    60   ~ 0
-a8
+a10
 Text Label 2230 3055 0    60   ~ 0
 a3
 Text Label 2230 3905 0    60   ~ 0
+a11
+Text Label 2230 4155 0    60   ~ 0
+a12
+Text Label 2230 4405 0    60   ~ 0
 a13
-Text Label 2230 4155 0    60   ~ 0
+Text Label 2230 4505 0    60   ~ 0
+a6
+Text Label 2230 4655 0    60   ~ 0
 a14
-Text Label 2230 4405 0    60   ~ 0
-a15
-Text Label 2230 4505 0    60   ~ 0
+Text Label 2230 4755 0    60   ~ 0
 a7
-Text Label 2230 4655 0    60   ~ 0
-a12
-Text Label 2230 4755 0    60   ~ 0
-a4
 Entry Wire Line
 	4580 2255 4680 2355
@@
 m0
 Text Label 4130 2505 0    60   ~ 0
+m1
+Text Label 4130 2755 0    60   ~ 0
+m2
+Text Label 4130 3005 0    60   ~ 0
+m3
+Text Label 4130 3955 0    60   ~ 0
+m4
+Text Label 4130 4205 0    60   ~ 0
 m5
-Text Label 4130 2755 0    60   ~ 0
-m4
-Text Label 4130 3005 0    60   ~ 0
+Text Label 4130 4455 0    60   ~ 0
 m6
-Text Label 4130 3955 0    60   ~ 0
-m1
-Text Label 4130 4205 0    60   ~ 0
-m3
-Text Label 4130 4455 0    60   ~ 0
+Text Label 4130 4705 0    60   ~ 0
 m7
-Text Label 4130 4705 0    60   ~ 0
-m2
 Text Label 6935 5555 0    60   ~ 0
 MultiplexedAddressBus
@@
 Connection ~ 7680 2555
 Text Label 2230 4255 0    60   ~ 0
-a6
+a5
 Text Label 2230 4005 0    60   ~ 0
-a5
+a4
 Wire Bus Line
 	5180 2355 5180 5705

Commit message: Finalize release
Parts:
- C1, C2, C3, C4: LCSC (none) -> C49678
- U2, U3: LCSC (none) -> C707097; Notes (none) -> HCT recommended, '157 works just as well
- U4, U5: Notes (none) -> Get from AliExpress
Changed lines of the file:
@@
 F 2 "Package_SO:SOIC-16_3.9x9.9mm_P1.27mm" H 3380 4455 50  0001 C CNN
 F 3 "" H 3380 4455 50  0001 C CNN
+F 4 "C707097" H 3380 4455 50  0001 C CNN "LCSC"
+F 5 "HCT recommended, '157 works just as well" H 3380 4455 50  0001 C CNN "Notes"
 	1    3380 4455
 	1    0    0    -1
@@
 F 2 "Package_DIP:DIP-18_W7.62mm_Socket_LongPads" H 6580 2755 50  0001 C CNN
 F 3 "DOCUMENTATION" H 6580 2755 50  0001 C CNN
+F 4 "Get from AliExpress" H 6580 2755 50  0001 C CNN "Notes"
 	1    6580 2755
 	1    0    0    -1
@@
 F 2 "Package_DIP:DIP-18_W7.62mm_Socket_LongPads" H 6580 4455 50  0001 C CNN
 F 3 "DOCUMENTATION" H 6580 4455 50  0001 C CNN
+F 4 "Get from AliExpress" H 6580 4455 50  0001 C CNN "Notes"
 	1    6580 4455
 	1    0    0    -1
@@
 F 2 "Package_SO:SOIC-16_3.9x9.9mm_P1.27mm" H 3380 2755 50  0001 C CNN
 F 3 "" H 3380 2755 50  0001 C CNN
+F 4 "C707097" H 3380 2755 50  0001 C CNN "LCSC"
+F 5 "HCT recommended, '157 works just as well" H 3380 2755 50  0001 C CNN "Notes"
 	1    3380 2755
 	1    0    0    -1
@@
 F 2 "Capacitor_SMD:C_0805_2012Metric_Pad1.18x1.45mm_HandSolder" H 3368 1205 50  0001 C CNN
 F 3 "~" H 3330 1355 50  0001 C CNN
+F 4 "C49678" H 3330 1355 50  0001 C CNN "LCSC"
 	1    3330 1355
 	1    0    0    -1
@@
 F 2 "Capacitor_SMD:C_0805_2012Metric_Pad1.18x1.45mm_HandSolder" H 6568 1055 50  0001 C CNN
 F 3 "~" H 6530 1205 50  0001 C CNN
+F 4 "C49678" H 6530 1205 50  0001 C CNN "LCSC"
 	1    6530 1205
 	1    0    0    -1
@@
 F 2 "Capacitor_SMD:C_0805_2012Metric_Pad1.18x1.45mm_HandSolder" H 3418 6255 50  0001 C CNN
 F 3 "~" H 3380 6405 50  0001 C CNN
+F 4 "C49678" H 3380 6405 50  0001 C CNN "LCSC"
 	1    3380 6405
 	1    0    0    -1
@@
 F 2 "Capacitor_SMD:C_0805_2012Metric_Pad1.18x1.45mm_HandSolder" H 6618 6255 50  0001 C CNN
 F 3 "~" H 6580 6405 50  0001 C CNN
+F 4 "C49678" H 6580 6405 50  0001 C CNN "LCSC"
 	1    6580 6405
 	1    0    0    -1
